File: elec/Control Board/Control v1/Adafruit-MAX31856-PCB-master.kicad_sch (KiCad schematic)
At the start: 5 parts, among them J10 MCP9600, J8 MCP9600, J9 MCP9600_

Commit message: Changes during team review.
Parts:
- added R108 (x3): DNI, Resistor_SMD:R_0603_1608Metric_Pad0.98x0.95mm_HandSolder, symbol Device:R
Connections:
- net GND: now also R108.1, R108.1, R108.1
- net at J10.9: now also R108.2
- net at J9.9: now also R108.2
- net at J8.9: now also R108.2
Other:
- note added: "TO DO: Solder on the modules directly to set subaddress. Default is 0x67."
