File: elec/Control Board/Control v1/Adafruit-MAX31850-thermocouple-breakout-board.kicad_sch (KiCad schematic)
At the start: 32 parts, among them J2 MAX31850K

Commit message: Changes during team review.
Parts:
- added R101: 1R0, Resistor_SMD:R_0603_1608Metric_Pad0.98x0.95mm_HandSolder, symbol Device:R
- added R203: 4K7, Resistor_SMD:R_0603_1608Metric_Pad0.98x0.95mm_HandSolder, symbol Device:R
- R101: value 1R0 -> DNI
Connections:
- net +VccMAX31850: now also R101.2, R203.2
- net DATA: now also R203.1
- new net +3V3_MAX31850K: R101.1
Other:
- note added: "Subaddress: 0x01 A0 Hi A1 Low A2 Low A3 Low"
- note added: "Subaddress: 0x02 A0 Low A1 Hi A2 Low A3 Low"
- note added: "Subaddress: 0x04 A0 Low A1 Low A2 Hi A3 Low"
- note removed: "Subaddess: 0x01 A0 Hi A1 Low A2 Low A3 Low"
- note removed: "Subaddess: 0x02 A0 Low A1 Hi A2 Low A3 Low"
- note removed: "Subaddess: 0x04 A0 Low A1 Low A2 Hi A3 Low"
Changed lines of the file:
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@@
   (junction (at 200.66 113.03) (diameter 0) (color 0 0 0 0)
   )
+  (junction (at 143.51 48.26) (diameter 0) (color 0 0 0 0)
+  )
+  (junction (at 143.51 135.89) (diameter 0) (color 0 0 0 0)
+  )
   (junction (at 29.21 78.74) (diameter 0) (color 0 0 0 0)
   )
@@
   (junction (at 50.8 166.37) (diameter 0) (color 0 0 0 0)
   )
+  (junction (at 43.18 29.21) (diameter 0) (color 0 0 0 0)
+  )
   (junction (at 100.33 48.26) (diameter 0) (color 0 0 0 0)
   )
@@
     (stroke (width 0) (type default))
   )
+  (wire (pts (xy 143.51 135.89) (xy 100.33 135.89))
+    (stroke (width 0) (type default))
+  )
   (wire (pts (xy 212.09 82.55) (xy 232.41 82.55))
     (stroke (width 0) (type default))
@@
     (stroke (width 0) (type default))
   )
+  (wire (pts (xy 43.18 29.21) (xy 43.18 40.64))
+    (stroke (width 0) (type default))
+  )
   (wire (pts (xy 111.76 175.26) (xy 111.76 171.45))
     (stroke (width 0) (type default))
@@
     (stroke (width 0) (type default))
   )
-  (wire (pts (xy 100.33 48.26) (xy 251.46 48.26))
+  (wire (pts (xy 143.51 128.27) (xy 143.51 135.89))
+    (stroke (width 0) (type default))
+  )
+  (wire (pts (xy 100.33 48.26) (xy 143.51 48.26))
     (stroke (width 0) (type default))
   )
@@
     (stroke (width 0) (type default))
   )
+  (wire (pts (xy 143.51 48.26) (xy 251.46 48.26))
+    (stroke (width 0) (type default))
+  )
   (wire (pts (xy 36.83 81.28) (xy 31.75 81.28))
     (stroke (width 0) (type default))
@@
     (stroke (width 0) (type default))
   )
-  (wire (pts (xy 43.18 24.13) (xy 43.18 40.64))
+  (wire (pts (xy 43.18 24.13) (xy 43.18 29.21))
     (stroke (width 0) (type default))
   )
@@
     (stroke (width 0) (type default))
   )
+  (wire (pts (xy 38.1 29.21) (xy 43.18 29.21))
+    (stroke (width 0) (type default))
+  )
   (wire (pts (xy 100.33 48.26) (xy 100.33 86.36))
     (stroke (width 0) (type default))
@@
     (stroke (width 0) (type default))
   )
+  (wire (pts (xy 27.94 29.21) (xy 30.48 29.21))
+    (stroke (width 0) (type default))
+  )
   (wire (pts (xy 95.25 148.59) (xy 132.08 148.59))
     (stroke (width 0) (type default))
   )
-  (wire (pts (xy 269.24 135.89) (xy 100.33 135.89))
+  (wire (pts (xy 269.24 135.89) (xy 143.51 135.89))
+    (stroke (width 0) (type default))
+  )
+  (wire (pts (xy 143.51 48.26) (xy 143.51 120.65))
     (stroke (width 0) (type default))
   )
@@
     )
   )
-  (text "Subaddess: 0x02\nA0 Low\nA1 Hi\nA2 Low\nA3 Low\n" (at 25.4 147.32 0)
+  (text "Subaddress: 0x02\nA0 Low\nA1 Hi\nA2 Low\nA3 Low\n" (at 25.4 147.32 0)
     (effects (font (size 1.27 1.27)) (justify left bottom))
   )
-  (text "Subaddess: 0x04\nA0 Low\nA1 Low\nA2 Hi\nA3 Low\n" (at 180.34 95.25 0)
+  (text "Subaddress: 0x04\nA0 Low\nA1 Low\nA2 Hi\nA3 Low\n" (at 180.34 95.25 0)
     (effects (font (size 1.27 1.27)) (justify left bottom))
   )
-  (text "Subaddess: 0x01\nA0 Hi\nA1 Low\nA2 Low\nA3 Low\n" (at 10.16 81.28 0)
+  (text "Subaddress: 0x01\nA0 Hi\nA1 Low\nA2 Low\nA3 Low\n" (at 10.16 81.28 0)
     (effects (font (size 1.27 1.27)) (justify left bottom))
   )
@@
     (effects (font (size 1.27 1.27)) (justify right))
   )
+  (hierarchical_label "+3V3_MAX31850K" (shape input) (at 27.94 29.21 180) (fields_autoplaced)
+    (effects (font (size 1.27 1.27)) (justify right))
+  )
   (hierarchical_label "DATA" (shape input) (at 80.01 101.6 180) (fields_autoplaced)
     (effects (font (size 1.2446 1.2446)) (justify right))
   )
+  (symbol (lib_id "Device:R") (at 34.29 29.21 90) (mirror x) (unit 1)
+    (in_bom yes) (on_board yes) (dnp no)
+    (property "Reference" "R101" (at 35.56 24.13 90)
+      (effects (font (size 1.27 1.27)))
+    )
+    (property "Value" "1R0" (at 34.29 26.67 90)
+      (effects (font (size 1.27 1.27)))
+    )
+    (property "Footprint" "Resistor_SMD:R_0603_1608Metric_Pad0.98x0.95mm_HandSolder" (at 34.29 27.432 90)
+      (effects (font (size 1.27 1.27)) hide)
+    )
+    (property "Datasheet" "~" (at 34.29 29.21 0)
+      (effects (font (size 1.27 1.27)) hide)
+    )
+    (property "Distributor 1" "JLCPCB" (at 34.29 29.21 90)
+      (effects (font (size 1.27 1.27)) hide)
+    )
+    (property "Distributor 1 PN" "C269434" (at 34.29 29.21 90)
+      (effects (font (size 1.27 1.27)) hide)
+    )
+    (property "Manufacturer" "TyoHM" (at 34.29 29.21 90)
+      (effects (font (size 1.27 1.27)) hide)
+    )
+    (property "MPN" "RMC060315%N" (at 34.29 29.21 90)
+      (effects (font (size 1.27 1.27)) hide)
+    )
+    (property "Description" "0.1W ±5% 1Ω 0603 Chip Resistor - Surface Mount ROHS" (at 34.29 29.21 0)
+      (effects (font (size 1.27 1.27)) hide)
+    )
+    (property "AssemblyType" "SMT" (at 34.29 29.21 0)
+      (effects (font (size 1.27 1.27)) hide)
+    )
+    (property "Cost" "0.0015" (at 34.29 29.21 0)
+      (effects (font (size 1.27 1.27)) hide)
+    )
+    (pin "1")
+    (pin "2")
+    (instances
+      (project "GeneralPurposeAlarmDevicePCB"
+        (path "/412a327d-1ee3-473e-bc00-1545004b7edf"
+          (reference "R101") (unit 1)
+        )
+      )
+      (project "Control v1"
+        (path "/c68c9deb-8d4d-42f0-adf8-4d3022f4ee59/0cb2f0dc-fe38-451d-b752-5d12a98f8d03"
+          (reference "R9") (unit 1)
+        )
+        (path "/c68c9deb-8d4d-42f0-adf8-4d3022f4ee59"
+          (reference "R51") (unit 1)
+        )
+        (path "/c68c9deb-8d4d-42f0-adf8-4d3022f4ee59/3ff32a52-b1ed-4756-8661-90a95f721605"
+          (reference "R82") (unit 1)
+        )
+      )
+    )
+  )
   (symbol (lib_id "Jumper:SolderJumper_3_Bridged12") (at 208.28 95.25 90) (mirror x) (unit 1)
     (in_bom yes) (on_board yes) (dnp no)
@@
       (effects (font (size 1.27 1.27)))
     )
-    (property "Value" "1R0" (at 35.56 38.1 90)
+    (property "Value" "DNI" (at 35.56 38.1 90)
       (effects (font (size 1.27 1.27)))
     )
@@
         )
       )
+    )
+  )
+  (symbol (lib_id "Device:R") (at 143.51 124.46 180) (unit 1)
+    (in_bom yes) (on_board yes) (dnp no)
+    (property "Reference" "R203" (at 148.59 123.19 0)
+      (effects (font (size 1.27 1.27)))
+    )
+    (property "Value" "4K7" (at 147.32 125.73 0)
+      (effects (font (size 1.27 1.27)))
+    )
+    (property "Footprint" "Resistor_SMD:R_0603_1608Metric_Pad0.98x0.95mm_HandSolder" (at 145.288 124.46 90)
+      (effects (font (size 1.27 1.27)) hide)
+    )
+    (property "Datasheet" "~" (at 143.51 124.46 0)
+      (effects (font (size 1.27 1.27)) hide)
+    )
+    (property "Distributor 1" "JLCPCB" (at 143.51 124.46 90)
+      (effects (font (size 1.27 1.27)) hide)
+    )
+    (property "Distributor 1 PN" "C269713" (at 143.51 124.46 90)
+      (effects (font (size 1.27 1.27)) hide)
+    )
+    (property "Manufacturer" "TyoHM" (at 143.51 124.46 90)
+      (effects (font (size 1.27 1.27)) hide)
+    )
+    (property "MPN" "RMC 0603 4K7 F N" (at 143.51 124.46 90)
+      (effects (font (size 1.27 1.27)) hide)
+    )
+    (property "Description" "1W ±1% 4.7kΩ 0603 Chip Resistor - Surface Mount ROHS" (at 143.51 124.46 0)
+      (effects (font (size 1.27 1.27)) hide)
+    )
+    (property "AssemblyType" "SMT" (at 143.51 124.46 0)
+      (effects (font (size 1.27 1.27)) hide)
+    )
+    (property "Cost" "0.0015" (at 143.51 124.46 0)
+      (effects (font (size 1.27 1.27)) hide)
+    )
+    (pin "1")
+    (pin "2")
+    (instances
+      (project "GeneralPurposeAlarmDevicePCB"
+        (path "/412a327d-1ee3-473e-bc00-1545004b7edf/00000000-0000-0000-0000-000062b3ac2f"
+          (reference "R203") (unit 1)
+        )
+      )
+      (project "Control v1"
+        (path "/c68c9deb-8d4d-42f0-adf8-4d3022f4ee59"
+          (reference "R77") (unit 1)
+        )
+        (path "/c68c9deb-8d4d-42f0-adf8-4d3022f4ee59/3ff32a52-b1ed-4756-8661-90a95f721605"
+          (reference "R83") (unit 1)
+        )
+      )

Commit message: Update parts in schematic for BOM generation.
Parts:
- J2, JP10, JP15: AssemblyType (none) -> HAND; Cost (none) -> 14.95; Distributor 1 (none) -> adafruit; Distributor 1 PN (none) -> 1727; MPN (none) -> 1727; Manufacturer (none) -> Adafruit
- JP6: AssemblyType (none) -> DNI; Cost (none) -> 0; Distributor 1 (none) -> PublicInvention; Distributor 1 PN (none) -> NA; MPN (none) -> NA; Manufacturer (none) -> NA
- R108: LongLead (none) -> NO
- TP103: Cost (none) -> NA
