File: elec/Control Board/Control v1/Adafruit-MAX31855-breakout-board.kicad_sch (KiCad schematic)
At the start: 5 parts

Commit message: Changes during team review.
Parts:
- added R101: 1R0, Resistor_SMD:R_0603_1608Metric_Pad0.98x0.95mm_HandSolder, symbol Device:R
- R101: value 1R0 -> DNI
Connections:
- net +VccMAX31855: now also R101.2
- new net +3V3_MAX31855: R101.1
Changed lines of the file:
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@@
 (kicad_sch (version 20230121) (generator eeschema)
   (paper "A4")
+  (junction (at 73.66 102.87) (diameter 0) (color 0 0 0 0)
+  )
   (junction (at 90.17 102.87) (diameter 0) (color 0 0 0 0)
   )
@@
     (stroke (width 0) (type default))
   )
+  (wire (pts (xy 46.99 83.82) (xy 60.96 83.82))
+    (stroke (width 0) (type default))
+  )
+  (wire (pts (xy 68.58 83.82) (xy 73.66 83.82))
+    (stroke (width 0) (type default))
+  )
+  (wire (pts (xy 73.66 83.82) (xy 73.66 102.87))
+    (stroke (width 0) (type default))
+  )
   (wire (pts (xy 95.25 116.84) (xy 95.25 133.35))
     (stroke (width 0) (type default))
@@
     (stroke (width 0) (type default))
   )
-  (wire (pts (xy 69.85 102.87) (xy 80.01 102.87))
+  (wire (pts (xy 73.66 102.87) (xy 80.01 102.87))
+    (stroke (width 0) (type default))
+  )
+  (wire (pts (xy 69.85 102.87) (xy 73.66 102.87))
     (stroke (width 0) (type default))
   )
@@
     (effects (font (size 1.27 1.27)) (justify right))
   )
+  (hierarchical_label "+3V3_MAX31855" (shape input) (at 46.99 83.82 180) (fields_autoplaced)
+    (effects (font (size 1.27 1.27)) (justify right))
+  )
   (symbol (lib_id "power:GND") (at 143.51 107.95 0) (unit 1)
     (in_bom yes) (on_board yes) (dnp no) (fields_autoplaced)
@@
     )
   )
+  (symbol (lib_id "Device:R") (at 64.77 83.82 90) (mirror x) (unit 1)
+    (in_bom yes) (on_board yes) (dnp no)
+    (property "Reference" "R101" (at 66.04 78.74 90)
+      (effects (font (size 1.27 1.27)))
+    )
+    (property "Value" "1R0" (at 64.77 81.28 90)
+      (effects (font (size 1.27 1.27)))
+    )
+    (property "Footprint" "Resistor_SMD:R_0603_1608Metric_Pad0.98x0.95mm_HandSolder" (at 64.77 82.042 90)
+      (effects (font (size 1.27 1.27)) hide)
+    )
+    (property "Datasheet" "~" (at 64.77 83.82 0)
+      (effects (font (size 1.27 1.27)) hide)
+    )
+    (property "Distributor 1" "JLCPCB" (at 64.77 83.82 90)
+      (effects (font (size 1.27 1.27)) hide)
+    )
+    (property "Distributor 1 PN" "C269434" (at 64.77 83.82 90)
+      (effects (font (size 1.27 1.27)) hide)
+    )
+    (property "Manufacturer" "TyoHM" (at 64.77 83.82 90)
+      (effects (font (size 1.27 1.27)) hide)
+    )
+    (property "MPN" "RMC060315%N" (at 64.77 83.82 90)
+      (effects (font (size 1.27 1.27)) hide)
+    )
+    (property "Description" "0.1W ±5% 1Ω 0603 Chip Resistor - Surface Mount ROHS" (at 64.77 83.82 0)
+      (effects (font (size 1.27 1.27)) hide)
+    )
+    (property "AssemblyType" "SMT" (at 64.77 83.82 0)
+      (effects (font (size 1.27 1.27)) hide)
+    )
+    (property "Cost" "0.0015" (at 64.77 83.82 0)
+      (effects (font (size 1.27 1.27)) hide)
+    )
+    (pin "1")
+    (pin "2")
+    (instances
+      (project "GeneralPurposeAlarmDevicePCB"
+        (path "/412a327d-1ee3-473e-bc00-1545004b7edf"
+          (reference "R101") (unit 1)
+        )
+      )
+      (project "Control v1"
+        (path "/c68c9deb-8d4d-42f0-adf8-4d3022f4ee59/0cb2f0dc-fe38-451d-b752-5d12a98f8d03"
+          (reference "R9") (unit 1)
+        )
+        (path "/c68c9deb-8d4d-42f0-adf8-4d3022f4ee59"
+          (reference "R51") (unit 1)
+        )
+        (path "/c68c9deb-8d4d-42f0-adf8-4d3022f4ee59/3ff32a52-b1ed-4756-8661-90a95f721605"
+          (reference "R7") (unit 1)
+        )
+        (path "/c68c9deb-8d4d-42f0-adf8-4d3022f4ee59/9d641288-e168-4964-816e-23e1814d1b66"
+          (reference "R84") (unit 1)
+        )
+      )
+    )
+  )
   (symbol (lib_id "power:GND") (at 77.47 109.22 0) (unit 1)
     (in_bom yes) (on_board yes) (dnp no)
@@
       (effects (font (size 1.27 1.27)))
     )
-    (property "Value" "1R0" (at 66.04 100.33 90)
+    (property "Value" "DNI" (at 66.04 100.33 90)
       (effects (font (size 1.27 1.27)))
     )

Commit message: Update parts in schematic for BOM generation.
Parts:
- JP1: AssemblyType (none) -> HAND; Cost (none) -> 14.95; Distributor 1 (none) -> adafruit; Distributor 1 PN (none) -> 269; MPN (none) -> 269; Manufacturer (none) -> Adafruit
- TP103: Cost (none) -> NA
Changed lines of the file:
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@@
       (effects (font (size 1.27 1.27)) hide)
     )
-    (property "Datasheet" "" (at 170.18 110.49 0)
+    (property "Datasheet" "https://www.adafruit.com/product/269" (at 170.18 110.49 0)
+      (effects (font (size 1.27 1.27)) hide)
+    )
+    (property "AssemblyType" "HAND" (at 170.18 110.49 0)
+      (effects (font (size 1.27 1.27)) hide)
+    )
+    (property "Cost" "14.95" (at 170.18 110.49 0)
+      (effects (font (size 1.27 1.27)) hide)
+    )
+    (property "Description" "Thermocouple Amplifier MAX31855 breakout board (MAX6675 upgrade)" (at 170.18 110.49 0)
+      (effects (font (size 1.27 1.27)) hide)
+    )
+    (property "Distributor 1" "adafruit" (at 170.18 110.49 0)
+      (effects (font (size 1.27 1.27)) hide)
+    )
+    (property "Distributor 1 PN" "269" (at 170.18 110.49 0)
+      (effects (font (size 1.27 1.27)) hide)
+    )
+    (property "MPN" "269" (at 170.18 110.49 0)
+      (effects (font (size 1.27 1.27)) hide)
+    )
+    (property "Manufacturer" "Adafruit" (at 170.18 110.49 0)
       (effects (font (size 1.27 1.27)) hide)
     )
@@
       (effects (font (size 1.27 1.27)) hide)
     )
-    (property "Datasheet" "" (at 137.16 110.49 0)
+    (property "Datasheet" "https://www.adafruit.com/product/269" (at 137.16 110.49 0)
+      (effects (font (size 1.27 1.27)) hide)
+    )
+    (property "AssemblyType" "HAND" (at 137.16 110.49 0)
+      (effects (font (size 1.27 1.27)) hide)
+    )
+    (property "Cost" "14.95" (at 137.16 110.49 0)
+      (effects (font (size 1.27 1.27)) hide)
+    )
+    (property "Description" "Thermocouple Amplifier MAX31855 breakout board (MAX6675 upgrade)" (at 137.16 110.49 0)
+      (effects (font (size 1.27 1.27)) hide)
+    )
+    (property "Distributor 1" "adafruit" (at 137.16 110.49 0)
+      (effects (font (size 1.27 1.27)) hide)
+    )
+    (property "Distributor 1 PN" "269" (at 137.16 110.49 0)
+      (effects (font (size 1.27 1.27)) hide)
+    )
+    (property "MPN" "269" (at 137.16 110.49 0)
+      (effects (font (size 1.27 1.27)) hide)
+    )
+    (property "Manufacturer" "Adafruit" (at 137.16 110.49 0)
       (effects (font (size 1.27 1.27)) hide)
     )
@@
       (effects (font (size 1.27 1.27)) hide)
     )
+    (property "Cost" "NA" (at 80.01 102.87 0)
+      (effects (font (size 1.27 1.27)) hide)
+    )
     (pin "1")
     (instances
@@
       (effects (font (size 1.27 1.27)) hide)
     )
-    (property "Datasheet" "" (at 104.14 111.76 0)
-      (effects (font (size 1.27 1.27)) hide)
-    )
+    (property "Datasheet" "https://www.adafruit.com/product/269" (at 104.14 111.76 0)
+      (effects (font (size 1.27 1.27)) hide)
+    )
+    (property "AssemblyType" "HAND" (at 104.14 111.76 0)
+      (effects (font (size 1.27 1.27)) hide)
+    )
+    (property "Cost" "14.95" (at 104.14 111.76 0)
+      (effects (font (size 1.27 1.27)) hide)
+    )
+    (property "Description" "Thermocouple Amplifier MAX31855 breakout board (MAX6675 upgrade)" (at 104.14 111.76 0)
+      (effects (font (size 1.27 1.27)) hide)
+    )
+    (property "Distributor 1" "adafruit" (at 104.14 111.76 0)
+      (effects (font (size 1.27 1.27)) hide)
+    )
+    (property "Distributor 1 PN" "269" (at 104.14 111.76 0)
+      (effects (font (size 1.27 1.27)) hide)
+    )
+    (property "MPN" "269" (at 104.14 111.76 0)
+      (effects (font (size 1.27 1.27)) hide)
+    )
+    (property "Manufacturer" "Adafruit" (at 104.14 111.76 0)
+      (effects (font (size 1.27 1.27)) hide)
+    )
