File: elec/Control Board/Control v1/SSR Interface.kicad_sch (KiCad schematic)
At the start: 3 parts, among them Q601 BSS138

Commit message: Changes during team review.
Parts:
- added R101: DNI, Resistor_SMD:R_0603_1608Metric_Pad0.98x0.95mm_HandSolder, symbol Device:R
- added R101: 1R0, Resistor_SMD:R_0603_1608Metric_Pad0.98x0.95mm_HandSolder, symbol Device:R
- added R102: 10K, Resistor_SMD:R_0603_1608Metric_Pad0.98x0.95mm_HandSolder, symbol Device:R
Connections:
- net +24V_SSR: now also R101.1
- net GND: now also R102.2
- net Heater: now also R102.1
- new net +12V_SSR: R101.1
- new net Heater_SSR_High: R101.2, R101.2

Commit message: Update parts in schematic for BOM generation.
Parts:
- R102: MPN RMC 0603 10K F N -> RMC060310KFN
- R108: LongLead (none) -> NO
Changed lines of the file:
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@@
       (effects (font (size 1.27 1.27)) hide)
     )
-    (property "Datasheet" "~" (at 62.23 69.85 0)
+    (property "Datasheet" "https://datasheet.lcsc.com/lcsc/1811101310_TyoHM-RMC06031K1-N_C269704.pdf" (at 62.23 69.85 0)
       (effects (font (size 1.27 1.27)) hide)
     )
@@
       (effects (font (size 1.27 1.27)) hide)
     )
-    (property "MPN" "RMC 0603 10K F N" (at 62.23 69.85 90)
+    (property "MPN" "RMC060310KFN" (at 62.23 69.85 90)
       (effects (font (size 1.27 1.27)) hide)
     )
-    (property "Description" "0.1W ±1% 10kΩ 0603  Chip Resistor - Surface Mount ROHS" (at 62.23 69.85 0)
+    (property "Description" "100mW ±1% 10kΩ 0603 Chip Resistor - Surface Mount ROHS" (at 62.23 69.85 0)
       (effects (font (size 1.27 1.27)) hide)
     )
@@
       (effects (font (size 1.27 1.27)) hide)
     )
-    (property "Datasheet" "~" (at 72.39 62.23 0)
+    (property "Datasheet" "https://datasheet.lcsc.com/lcsc/1811101310_TyoHM-RMC06031K1-N_C269704.pdf" (at 72.39 62.23 0)
       (effects (font (size 1.27 1.27)) hide)
     )
@@
       (effects (font (size 1.27 1.27)) hide)
     )
+    (property "LongLead" "NO" (at 72.39 62.23 0)
+      (effects (font (size 1.27 1.27)) hide)
+    )
