File: elec/Control Board/Control v1/Fan controller.kicad_sch (KiCad schematic)
At the start: 37 parts, among them J10 Conn_01x05, J11 Conn_01x04, J12 Conn_01x07, J20 Conn_01x04, J6 DB25_Female_MountingHoles, J9 Conn_01x04, Q2 NCE01P30K, Q601 BSS138

Commit message: Changes during team review.
Parts:
- removed R7: DNI, Resistor_SMD:R_0603_1608Metric_Pad0.98x0.95mm_HandSolder, symbol Device:R
- added R90: DNI, Resistor_SMD:R_0603_1608Metric_Pad0.98x0.95mm_HandSolder, symbol Device:R
Connections:
- net +24VFan: now also R90.1
- net GND: now also J6.14 (P14), J6.15 (P15), J6.16 (P16), J6.17 (P17)
- net Switched_Fan_Power: now also R90.2
- net TachFan1: no longer J6.14 (P14), J6.15 (P15), J6.16 (P16), J6.17 (P17)
Other:
- note added: "This resistor keeps the fan OFF at power up."
- moved on the sheet: C104
Changed lines of the file:
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@@
   (junction (at 36.83 53.34) (diameter 0) (color 0 0 0 0)
   )
-  (junction (at 52.07 104.14) (diameter 0) (color 0 0 0 0)
-  )
   (junction (at 54.61 111.76) (diameter 0) (color 0 0 0 0)
   )
@@
   (junction (at 33.02 149.86) (diameter 0) (color 0 0 0 0)
   )
+  (junction (at 207.01 30.48) (diameter 0) (color 0 0 0 0)
+  )
   (junction (at 167.64 60.96) (diameter 0) (color 0 0 0 0)
   )
@@
   (junction (at 46.99 93.98) (diameter 0) (color 0 0 0 0)
   )
+  (junction (at 52.07 104.14) (diameter 0) (color 0 0 0 0)
+  )
   (junction (at 54.61 106.68) (diameter 0) (color 0 0 0 0)
   )
@@
   (junction (at 49.53 99.06) (diameter 0) (color 0 0 0 0)
   )
-  (junction (at 81.28 121.92) (diameter 0) (color 0 0 0 0)
+  (junction (at 207.01 66.04) (diameter 0) (color 0 0 0 0)
   )
-  (junction (at 52.07 111.76) (diameter 0) (color 0 0 0 0)
+  (junction (at 81.28 121.92) (diameter 0) (color 0 0 0 0)
   )
   (junction (at 200.66 124.46) (diameter 0) (color 0 0 0 0)
@@
     (stroke (width 0) (type default))
   )
-  (wire (pts (xy 52.07 104.14) (xy 93.98 104.14))
+  (wire (pts (xy 39.37 104.14) (xy 52.07 104.14))
     (stroke (width 0) (type default))
   )
@@
     (stroke (width 0) (type default))
   )
-  (wire (pts (xy 161.29 66.04) (xy 229.87 66.04))
+  (wire (pts (xy 161.29 66.04) (xy 207.01 66.04))
     (stroke (width 0) (type default))
   )
@@
     (stroke (width 0) (type default))
   )
-  (wire (pts (xy 69.85 115.57) (xy 64.77 115.57))
+  (wire (pts (xy 64.77 115.57) (xy 85.09 115.57))
     (stroke (width 0) (type default))
   )
@@
     (stroke (width 0) (type default))
   )
+  (wire (pts (xy 207.01 66.04) (xy 229.87 66.04))
+    (stroke (width 0) (type default))
+  )
   (wire (pts (xy 85.09 54.61) (xy 118.11 54.61))
     (stroke (width 0) (type default))
@@
     (stroke (width 0) (type default))
   )
-  (wire (pts (xy 52.07 111.76) (xy 52.07 137.16))
-    (stroke (width 0) (type default))
-  )
   (wire (pts (xy 33.02 130.81) (xy 46.99 130.81))
     (stroke (width 0) (type default))
@@
     (stroke (width 0) (type default))
   )
-  (wire (pts (xy 151.13 30.48) (xy 229.87 30.48))
+  (wire (pts (xy 151.13 30.48) (xy 207.01 30.48))
     (stroke (width 0) (type default))
   )
@@
     (stroke (width 0) (type default))
   )
-  (wire (pts (xy 39.37 104.14) (xy 52.07 104.14))
+  (wire (pts (xy 255.27 57.15) (xy 255.27 54.61))
     (stroke (width 0) (type default))
   )
-  (wire (pts (xy 255.27 57.15) (xy 255.27 54.61))
+  (wire (pts (xy 52.07 104.14) (xy 52.07 137.16))
     (stroke (width 0) (type default))
   )
@@
     (stroke (width 0) (type default))
   )
-  (wire (pts (xy 39.37 111.76) (xy 52.07 111.76))
+  (wire (pts (xy 39.37 111.76) (xy 54.61 111.76))
     (stroke (width 0) (type default))
   )
@@
     (stroke (width 0) (type default))
   )
-  (wire (pts (xy 52.07 111.76) (xy 54.61 111.76))
-    (stroke (width 0) (type default))
-  )
   (wire (pts (xy 111.76 64.77) (xy 118.11 64.77))
     (stroke (width 0) (type default))
@@
     (stroke (width 0) (type default))
   )
+  (wire (pts (xy 52.07 104.14) (xy 93.98 104.14))
+    (stroke (width 0) (type default))
+  )
   (wire (pts (xy 189.23 71.12) (xy 185.42 71.12))
     (stroke (width 0) (type default))
@@
     (stroke (width 0) (type default))
   )
-  (wire (pts (xy 33.02 142.24) (xy 33.02 130.81))
+  (wire (pts (xy 33.02 137.16) (xy 33.02 130.81))
     (stroke (width 0) (type default))
   )
@@
     (stroke (width 0) (type default))
   )
-  (wire (pts (xy 77.47 115.57) (xy 85.09 115.57))
-    (stroke (width 0) (type default))
-  )
   (wire (pts (xy 275.59 73.66) (xy 275.59 76.2))
     (stroke (width 0) (type default))
@@
     (stroke (width 0) (type default))
   )
-  (wire (pts (xy 52.07 111.76) (xy 52.07 104.14))
-    (stroke (width 0) (type default))
-  )
   (wire (pts (xy 266.7 62.23) (xy 262.89 62.23))
     (stroke (width 0) (type default))
@@
     (stroke (width 0) (type default))
   )
+  (wire (pts (xy 207.01 57.15) (xy 207.01 66.04))
+    (stroke (width 0) (type default))
+  )
   (wire (pts (xy 229.87 44.45) (xy 229.87 49.53))
     (stroke (width 0) (type default))
@@
     (stroke (width 0) (type default))
   )
+  (wire (pts (xy 207.01 30.48) (xy 229.87 30.48))
+    (stroke (width 0) (type default))
+  )
   (wire (pts (xy 167.64 54.61) (xy 167.64 60.96))
     (stroke (width 0) (type default))
@@
     (stroke (width 0) (type default))
   )
+  (wire (pts (xy 33.02 144.78) (xy 33.02 149.86))
+    (stroke (width 0) (type default))
+  )
   (wire (pts (xy 59.69 114.3) (xy 59.69 121.92))
     (stroke (width 0) (type default))
@@
     (stroke (width 0) (type default))
   )
+  (wire (pts (xy 207.01 49.53) (xy 207.01 30.48))
+    (stroke (width 0) (type default))
+  )
   (wire (pts (xy 39.37 76.2) (xy 87.63 76.2))
     (stroke (width 0) (type default))
@@
     (effects (font (size 1.27 1.27) (thickness 0.254) bold) (justify left bottom))
   )
+  (text "This resistor keeps the fan OFF at power up." (at 246.38 95.25 0)
+    (effects (font (size 1.27 1.27)) (justify left bottom))
+  )
   (label "TachFan4" (at 67.31 111.76 0) (fields_autoplaced)
     (effects (font (size 1.27 1.27)) (justify left bottom))
@@
     )
   )
-  (symbol (lib_id "Device:R") (at 73.66 115.57 90) (unit 1)
-    (in_bom yes) (on_board yes) (dnp no)
-    (property "Reference" "R7" (at 69.85 113.03 90)
-      (effects (font (size 1.27 1.27)))
-    )
-    (property "Value" "DNI" (at 77.47 113.03 90)
-      (effects (font (size 1.27 1.27)))
-    )
-    (property "Footprint" "Resistor_SMD:R_0603_1608Metric_Pad0.98x0.95mm_HandSolder" (at 73.66 117.348 90)
-      (effects (font (size 1.27 1.27)) hide)
-    )
-    (property "Datasheet" "~" (at 73.66 115.57 0)
-      (effects (font (size 1.27 1.27)) hide)
-    )
-    (property "AssemblyType" "SMT" (at 73.66 115.57 0)
-      (effects (font (size 1.27 1.27)) hide)
-    )
-    (property "Distributor 1" "NA" (at 73.66 115.57 0)
-      (effects (font (size 1.27 1.27)) hide)
-    )
-    (property "Distributor 1 PN" "NA" (at 73.66 115.57 0)
-      (effects (font (size 1.27 1.27)) hide)
-    )
-    (property "Cost" "0.0015" (at 73.66 115.57 0)
-      (effects (font (size 1.27 1.27)) hide)
-    )
-    (property "LongLead" "NO" (at 73.66 115.57 0)
-      (effects (font (size 1.27 1.27)) hide)
-    )
-    (property "Description" "Do Not Insert" (at 73.66 115.57 0)
-      (effects (font (size 1.27 1.27)) hide)
-    )
-    (pin "1")
-    (pin "2")
-    (instances
-      (project "Control v1"
-        (path "/c68c9deb-8d4d-42f0-adf8-4d3022f4ee59"
-          (reference "R7") (unit 1)
-        )
-        (path "/c68c9deb-8d4d-42f0-adf8-4d3022f4ee59/0cb2f0dc-fe38-451d-b752-5d12a98f8d03"
-          (reference "R32") (unit 1)
-        )
-      )
-    )
-  )
   (symbol (lib_id "power:GND") (at 275.59 76.2 0) (mirror y) (unit 1)
     (in_bom yes) (on_board yes) (dnp no) (fields_autoplaced)
@@
     )
   )
-  (symbol (lib_id "Device:C") (at 33.02 146.05 0) (mirror y) (unit 1)
+  (symbol (lib_id "Device:C") (at 33.02 140.97 0) (mirror y) (unit 1)
     (in_bom yes) (on_board yes) (dnp no)
-    (property "Reference" "C104" (at 30.099 144.8816 0)
+    (property "Reference" "C104" (at 30.099 139.8016 0)
       (effects (font (size 1.27 1.27)) (justify left))
     )
-    (property "Value" "39pF" (at 30.099 147.193 0)
+    (property "Value" "39pF" (at 30.099 142.113 0)
       (effects (font (size 1.27 1.27)) (justify left))
     )
-    (property "Footprint" "Capacitor_SMD:C_0603_1608Metric_Pad1.08x0.95mm_HandSolder" (at 32.0548 149.86 0)
+    (property "Footprint" "Capacitor_SMD:C_0603_1608Metric_Pad1.08x0.95mm_HandSolder" (at 32.0548 144.78 0)
       (effects (font (size 1.27 1.27)) hide)
     )
-    (property "Datasheet" "~" (at 33.02 146.05 0)
+    (property "Datasheet" "~" (at 33.02 140.97 0)
       (effects (font (size 1.27 1.27)) hide)
     )
-    (property "AssemblyType" "SMT" (at 33.02 146.05 0)
+    (property "AssemblyType" "SMT" (at 33.02 140.97 0)
       (effects (font (size 1.27 1.27)) hide)
     )
-    (property "Distributor 1" "JLCPCB" (at 33.02 146.05 0)
+    (property "Distributor 1" "JLCPCB" (at 33.02 140.97 0)
       (effects (font (size 1.27 1.27)) hide)
     )
-    (property "Distributor 1 PN" "C107049" (at 33.02 146.05 0)
+    (property "Distributor 1 PN" "C107049" (at 33.02 140.97 0)
       (effects (font (size 1.27 1.27)) hide)
     )
-    (property "MPN" "CC0603JRNPO9BN390" (at 33.02 146.05 0)
+    (property "MPN" "CC0603JRNPO9BN390" (at 33.02 140.97 0)
       (effects (font (size 1.27 1.27)) hide)
     )
-    (property "Manufacturer" "YAGEO" (at 33.02 146.05 0)
+    (property "Manufacturer" "YAGEO" (at 33.02 140.97 0)
       (effects (font (size 1.27 1.27)) hide)
     )
-    (property "Cost" "0.003" (at 33.02 146.05 0)
+    (property "Cost" "0.003" (at 33.02 140.97 0)
       (effects (font (size 1.27 1.27)) hide)
     )
@@
         )
       )
+    )
+  )
+  (symbol (lib_id "Device:R") (at 207.01 53.34 0) (mirror y) (unit 1)
+    (in_bom yes) (on_board yes) (dnp no) (fields_autoplaced)
+    (property "Reference" "R90" (at 204.47 52.705 0)
+      (effects (font (size 1.27 1.27)) (justify left))
+    )
+    (property "Value" "DNI" (at 204.47 55.245 0)
+      (effects (font (size 1.27 1.27)) (justify left))
+    )
+    (property "Footprint" "Resistor_SMD:R_0603_1608Metric_Pad0.98x0.95mm_HandSolder" (at 208.788 53.34 90)
+      (effects (font (size 1.27 1.27)) hide)
+    )
+    (property "Datasheet" "~" (at 207.01 53.34 0)
+      (effects (font (size 1.27 1.27)) hide)
+    )
+    (pin "1")
+    (pin "2")
+    (instances
+      (project "Control v1"
+        (path "/c68c9deb-8d4d-42f0-adf8-4d3022f4ee59/0cb2f0dc-fe38-451d-b752-5d12a98f8d03"
+          (reference "R90") (unit 1)
+        )
+      )

Commit message: Lots of routing. Lots remaining.
Connections:
- net LOOPBACK25: now reaches J11.3 (Pin_3), J6.25 (P25)
- net LOOPBACK13: now reaches J11.4 (Pin_4), J6.13
Other:
- note added: "Loop back signals DB 25 and 13 Due pins ?? ???"
- note removed: "Loop back signals DB 24 and 13 Due pins ?? ???"
Changed lines of the file:
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@@
   (junction (at 187.96 124.46) (diameter 0) (color 0 0 0 0)
   )
+  (junction (at 104.14 80.01) (diameter 0) (color 0 0 0 0)
+  )
   (junction (at 63.5 45.72) (diameter 0) (color 0 0 0 0)
   )
@@
   (junction (at 44.45 88.9) (diameter 0) (color 0 0 0 0)
   )
+  (junction (at 100.33 82.55) (diameter 0) (color 0 0 0 0)
+  )
   (junction (at 63.5 78.74) (diameter 0) (color 0 0 0 0)
   )
@@
     (stroke (width 0) (type default))
   )
+  (wire (pts (xy 93.98 82.55) (xy 100.33 82.55))
+    (stroke (width 0) (type default))
+  )
   (wire (pts (xy 60.96 62.23) (xy 118.11 62.23))
     (stroke (width 0) (type default))
@@
     (stroke (width 0) (type default))
   )
+  (wire (pts (xy 93.98 80.01) (xy 104.14 80.01))
+    (stroke (width 0) (type default))
+  )
   (wire (pts (xy 199.39 69.85) (xy 199.39 86.36))
     (stroke (width 0) (type default))
@@
     (effects (font (size 1.27 1.27)) (justify left bottom))
   )
-  (text "Loop back signals\nDB 24 and 13\nDue pins ?? ???" (at 115.57 83.82 0)
+  (text "Loop back signals\nDB 25 and 13\nDue pins ?? ???" (at 115.57 83.82 0)
     (effects (font (size 1.27 1.27)) (justify left bottom))
   )
@@
     (effects (font (size 1.27 1.27)) (justify right))
   )
+  (hierarchical_label "LOOPBACK13" (shape input) (at 93.98 80.01 180) (fields_autoplaced)
+    (effects (font (size 1.27 1.27)) (justify right))
+  )
   (hierarchical_label "+5VFan" (shape input) (at 186.69 111.76 180) (fields_autoplaced)
     (effects (font (size 1.27 1.27)) (justify right))
   )
+  (hierarchical_label "LOOPBACK25" (shape input) (at 93.98 82.55 180) (fields_autoplaced)
+    (effects (font (size 1.27 1.27)) (justify right))
+  )

Commit message: Update parts in schematic for BOM generation.
Parts:
- D1, D2: Cost (none) -> 1000000
- J10: Cost (none) -> 0.0791; Distributor 1 (none) -> JLCPCB; Distributor 1 PN (none) -> C2897368; MPN (none) -> PM254-1-05-Z-8.5; Manufacturer (none) -> HCTL
- J11, J20, J9: Cost (none) -> 0.0342; Distributor 1 (none) -> JLCPCB; Distributor 1 PN (none) -> C2905415; MPN (none) -> KH-2.54FH-1X4P-H8.5; Manufacturer (none) -> Shenzhen Kinghelm Elec
- J12: Cost (none) -> 0.0543; Distributor 1 (none) -> JLCPCB; Distributor 1 PN (none) -> C2932672
- J6: AssemblyType (none) -> HAND; Cost (none) -> 0.7217; Distributor 1 (none) -> JLCPCB; Distributor 1 PN (none) -> C190083; MPN (none) -> D-DMR025PF-D002; Manufacturer (none) -> Ckmtw(Shenzhen Cankemeng)
- R102: MPN RMC 0603 10K F N -> RMC060310KFN
- R108: LongLead (none) -> NO
- R34, R35, R43, R90: Cost (none) -> 0.0015
- R39, R40: LongLead (none) -> NO; MPN (none) -> RMC060310KFN; Manufacturer (none) -> TyoHM
- TP103: Cost (none) -> NA

Commit message: Add BOM spread sheet and a JLCPCB BOM.
Parts:
- C104: LongLead (none) -> NO
Changed lines of the file:
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@@
       (effects (font (size 1.27 1.27)) hide)
     )
-    (property "Datasheet" "~" (at 81.28 133.35 0)
+    (property "Datasheet" "https://datasheet.lcsc.com/lcsc/1811082118_YAGEO-CC0603JRNPO9BN390_C107049.pdf" (at 81.28 133.35 0)
       (effects (font (size 1.27 1.27)) hide)
     )
@@
     )
     (property "Cost" "0.003" (at 81.28 133.35 0)
+      (effects (font (size 1.27 1.27)) hide)
+    )
+    (property "Description" "50V 39pF NP0 ±5% 0603 Multilayer Ceramic Ca" (at 81.28 133.35 0)
+      (effects (font (size 1.27 1.27)) hide)
+    )
+    (property "LongLead" "NO" (at 81.28 133.35 0)
       (effects (font (size 1.27 1.27)) hide)
     )
@@
       (effects (font (size 1.27 1.27)) hide)
     )
-    (property "Datasheet" "~" (at 67.31 133.35 0)
+    (property "Datasheet" "https://datasheet.lcsc.com/lcsc/1811082118_YAGEO-CC0603JRNPO9BN390_C107049.pdf" (at 67.31 133.35 0)
       (effects (font (size 1.27 1.27)) hide)
     )
@@
     )
     (property "Cost" "0.003" (at 67.31 133.35 0)
+      (effects (font (size 1.27 1.27)) hide)
+    )
+    (property "Description" "50V 39pF NP0 ±5% 0603 Multilayer Ceramic Ca" (at 67.31 133.35 0)
+      (effects (font (size 1.27 1.27)) hide)
+    )
+    (property "LongLead" "NO" (at 67.31 133.35 0)
       (effects (font (size 1.27 1.27)) hide)
     )
@@
       (effects (font (size 1.27 1.27)) hide)
     )
-    (property "Datasheet" "~" (at 72.39 140.97 0)
+    (property "Datasheet" "https://datasheet.lcsc.com/lcsc/1811082118_YAGEO-CC0603JRNPO9BN390_C107049.pdf" (at 72.39 140.97 0)
       (effects (font (size 1.27 1.27)) hide)
     )
@@
     )
     (property "Cost" "0.003" (at 72.39 140.97 0)
+      (effects (font (size 1.27 1.27)) hide)
+    )
+    (property "Description" "50V 39pF NP0 ±5% 0603 Multilayer Ceramic Ca" (at 72.39 140.97 0)
+      (effects (font (size 1.27 1.27)) hide)
+    )
+    (property "LongLead" "NO" (at 72.39 140.97 0)
       (effects (font (size 1.27 1.27)) hide)
     )
@@
       (effects (font (size 1.27 1.27)) hide)
     )
-    (property "Datasheet" "~" (at 43.18 135.89 0)
+    (property "Datasheet" "https://datasheet.lcsc.com/lcsc/1811082118_YAGEO-CC0603JRNPO9BN390_C107049.pdf" (at 43.18 135.89 0)
       (effects (font (size 1.27 1.27)) hide)
     )
@@
     )
     (property "Cost" "0.003" (at 43.18 135.89 0)
+      (effects (font (size 1.27 1.27)) hide)
+    )
+    (property "Description" "50V 39pF NP0 ±5% 0603 Multilayer Ceramic Ca" (at 43.18 135.89 0)
+      (effects (font (size 1.27 1.27)) hide)
+    )
+    (property "LongLead" "NO" (at 43.18 135.89 0)
       (effects (font (size 1.27 1.27)) hide)
     )
@@
       (effects (font (size 1.27 1.27)) hide)
     )
-    (property "Datasheet" "~" (at 17.78 140.97 0)
+    (property "Datasheet" "https://datasheet.lcsc.com/lcsc/1811082118_YAGEO-CC0603JRNPO9BN390_C107049.pdf" (at 17.78 140.97 0)
       (effects (font (size 1.27 1.27)) hide)
     )
@@
     )
     (property "Cost" "0.003" (at 17.78 140.97 0)
+      (effects (font (size 1.27 1.27)) hide)
+    )
+    (property "Description" "50V 39pF NP0 ±5% 0603 Multilayer Ceramic Ca" (at 17.78 140.97 0)
+      (effects (font (size 1.27 1.27)) hide)
+    )
+    (property "LongLead" "NO" (at 17.78 140.97 0)
       (effects (font (size 1.27 1.27)) hide)
     )
@@
       (effects (font (size 1.27 1.27)) hide)
     )
-    (property "Datasheet" "~" (at 52.07 140.97 0)
+    (property "Datasheet" "https://datasheet.lcsc.com/lcsc/1811082118_YAGEO-CC0603JRNPO9BN390_C107049.pdf" (at 52.07 140.97 0)
       (effects (font (size 1.27 1.27)) hide)
     )
@@
     )
     (property "Cost" "0.003" (at 52.07 140.97 0)
+      (effects (font (size 1.27 1.27)) hide)
+    )
+    (property "Description" "50V 39pF NP0 ±5% 0603 Multilayer Ceramic Ca" (at 52.07 140.97 0)
+      (effects (font (size 1.27 1.27)) hide)
+    )
+    (property "LongLead" "NO" (at 52.07 140.97 0)
       (effects (font (size 1.27 1.27)) hide)
     )
@@
       (effects (font (size 1.27 1.27)) hide)
     )
-    (property "Datasheet" "~" (at 33.02 140.97 0)
+    (property "Datasheet" "https://datasheet.lcsc.com/lcsc/1811082118_YAGEO-CC0603JRNPO9BN390_C107049.pdf" (at 33.02 140.97 0)
       (effects (font (size 1.27 1.27)) hide)
     )
@@
     )
     (property "Cost" "0.003" (at 33.02 140.97 0)
+      (effects (font (size 1.27 1.27)) hide)
+    )
+    (property "Description" "50V 39pF NP0 ±5% 0603 Multilayer Ceramic Ca" (at 33.02 140.97 0)
+      (effects (font (size 1.27 1.27)) hide)
+    )
+    (property "LongLead" "NO" (at 33.02 140.97 0)
       (effects (font (size 1.27 1.27)) hide)
     )
@@
       (effects (font (size 1.27 1.27)) hide)
     )
-    (property "Datasheet" "~" (at 25.4 52.07 0)
+    (property "Datasheet" "https://datasheet.lcsc.com/lcsc/1811082118_YAGEO-CC0603JRNPO9BN390_C107049.pdf" (at 25.4 52.07 0)
       (effects (font (size 1.27 1.27)) hide)
     )
@@
     )
     (property "Cost" "0.003" (at 25.4 52.07 0)
+      (effects (font (size 1.27 1.27)) hide)
+    )
+    (property "Description" "50V 39pF NP0 ±5% 0603 Multilayer Ceramic Ca" (at 25.4 52.07 0)
+      (effects (font (size 1.27 1.27)) hide)
+    )
+    (property "LongLead" "NO" (at 25.4 52.07 0)
       (effects (font (size 1.27 1.27)) hide)
     )
@@
       (effects (font (size 1.27 1.27)) hide)
     )
-    (property "Datasheet" "~" (at 91.44 140.97 0)
+    (property "Datasheet" "https://datasheet.lcsc.com/lcsc/1811082118_YAGEO-CC0603JRNPO9BN390_C107049.pdf" (at 91.44 140.97 0)
       (effects (font (size 1.27 1.27)) hide)
     )
@@
       (effects (font (size 1.27 1.27)) hide)
     )
+    (property "Description" "50V 39pF NP0 ±5% 0603 Multilayer Ceramic Ca" (at 91.44 140.97 0)
+      (effects (font (size 1.27 1.27)) hide)
+    )
+    (property "LongLead" "NO" (at 91.44 140.97 0)
+      (effects (font (size 1.27 1.27)) hide)
+    )
