File: elec/Control Board/Control_1v1/Control_1v1/Adafruit-MAX31855-breakout-board.kicad_sch (KiCad schematic)
At the start: 6 parts

Commit message: Add sheet with title block.
Other:
- company: (none) -> Public Invention
- title: (none) -> Control Interconnect Board

Commit message: Fix J10 backwards.
Other:
- title: Control Interconnect Board -> Control Interconnect Board OEDCS
Changed lines of the file:
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@@
   (paper "USLedger")
   (title_block
-    (title "Control Interconnect Board")
+    (title "Control Interconnect Board OEDCS")
     (date "2023-10-10")
     (rev "Rev 1.1")
     (company "Public Invention")
-    (comment 1 "Contributor: Lawrence Kinceloe")
+    (comment 1 "GNU Affero General Public License v3.0")
+    (comment 2 "Contributor: Lawrence Kinceloe")
+    (comment 3 "Drawn By: (Forrest) Lee Erickson")
   )
   (junction (at 73.66 102.87) (diameter 0) (color 0 0 0 0)

Commit message: Add power shutdown button. Add thermocouple ground screw terminals. Isolate SCL from SDA traces. Make first cut BOM.
Parts:
- R101: LongLead (none) -> NO
Changed lines of the file:
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@@
+      (effects (font (size 1.27 1.27)) hide)
+    )
+    (property "LongLead" "NO" (at 64.77 83.82 0)
       (effects (font (size 1.27 1.27)) hide)
     )
