File: elec/Control Board/Control_1v1/Control_1v1/Adafruit-MAX31855-breakout-board.kicad_sch (KiCad schematic)
At the start: 6 parts

Commit message: Changes to change headders to sockets. Scockets for thermcouple amplifiers.
Parts:
- JP1: Distributor 1 adafruit -> JLCPCB; Distributor 1 PN 269 -> C2905416
Changed lines of the file:
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@@
       (effects (font (size 1.27 1.27)) hide)
     )
-    (property "Description" "Thermocouple Amplifier MAX31855 breakout board (MAX6675 upgrade)" (at 170.18 110.49 0)
-      (effects (font (size 1.27 1.27)) hide)
-    )
-    (property "Distributor 1" "adafruit" (at 170.18 110.49 0)
-      (effects (font (size 1.27 1.27)) hide)
-    )
-    (property "Distributor 1 PN" "269" (at 170.18 110.49 0)
+    (property "Description" "2.54mm Plugin 3A 6P -40℃~+105℃ Straight 1x6P 8.5mm Top Square Holes Plugin,P=2.54mm Female Headers ROHS" (at 170.18 110.49 0)
+      (effects (font (size 1.27 1.27)) hide)
+    )
+    (property "Distributor 1" "JLCPCB" (at 170.18 110.49 0)
+      (effects (font (size 1.27 1.27)) hide)
+    )
+    (property "Distributor 1 PN" "C2905416" (at 170.18 110.49 0)
       (effects (font (size 1.27 1.27)) hide)
     )
@@
       (effects (font (size 1.27 1.27)) hide)
     )
-    (property "Description" "Thermocouple Amplifier MAX31855 breakout board (MAX6675 upgrade)" (at 137.16 110.49 0)
-      (effects (font (size 1.27 1.27)) hide)
-    )
-    (property "Distributor 1" "adafruit" (at 137.16 110.49 0)
-      (effects (font (size 1.27 1.27)) hide)
-    )
-    (property "Distributor 1 PN" "269" (at 137.16 110.49 0)
+    (property "Description" "2.54mm Plugin 3A 6P -40℃~+105℃ Straight 1x6P 8.5mm Top Square Holes Plugin,P=2.54mm Female Headers ROHS" (at 137.16 110.49 0)
+      (effects (font (size 1.27 1.27)) hide)
+    )
+    (property "Distributor 1" "JLCPCB" (at 137.16 110.49 0)
+      (effects (font (size 1.27 1.27)) hide)
+    )
+    (property "Distributor 1 PN" "C2905416" (at 137.16 110.49 0)
       (effects (font (size 1.27 1.27)) hide)
     )
@@
       (effects (font (size 1.27 1.27)) hide)
     )
-    (property "Description" "Thermocouple Amplifier MAX31855 breakout board (MAX6675 upgrade)" (at 104.14 111.76 0)
-      (effects (font (size 1.27 1.27)) hide)
-    )
-    (property "Distributor 1" "adafruit" (at 104.14 111.76 0)
-      (effects (font (size 1.27 1.27)) hide)
-    )
-    (property "Distributor 1 PN" "269" (at 104.14 111.76 0)
-      (effects (font (size 1.27 1.27)) hide)
-    )
+    (property "Description" "2.54mm Plugin 3A 6P -40℃~+105℃ Straight 1x6P 8.5mm Top Square Holes Plugin,P=2.54mm Female Headers ROHS" (at 104.14 111.76 0)
+      (effects (font (size 1.27 1.27)) hide)
+    )
+    (property "Distributor 1" "JLCPCB" (at 104.14 111.76 0)
+      (effects (font (size 1.27 1.27)) hide)
+    )
+    (property "Distributor 1 PN" "C2905416" (at 104.14 111.76 0)
+      (effects (font (size 1.27 1.27)) hide)
+    )
