File: elec/Control Board/Control_1v1/Control_1v1/I2C_Level_Shifter.kicad_sch (KiCad schematic)
At the start: 21 parts, among them J201 0.100_2Pin, J202 Conn_01x04, Q201 BSS138, Q202 BSS138

Commit message: Move components away from J35, J36.
Parts:
- J202: Distributor 1 PN C2905415 -> C6332197; MPN KH-2.54FH-1X4P-H8.5 -> HB-PH3-25414PB2GOP; Manufacturer Shenzhen Kinghelm Elec -> Hanbo Electronic
Changed lines of the file:
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@@
       (effects (font (size 1.27 1.27)) hide)
     )
-    (property "Datasheet" "KH-2.54FH-1X4P-H8.5.pdf" (at 293.37 129.54 0)
+    (property "Datasheet" "HB-PH3-25414PB2GOP.pdf" (at 293.37 129.54 0)
       (effects (font (size 1.27 1.27)) hide)
     )
@@
       (effects (font (size 1.27 1.27)) hide)
     )
-    (property "Distributor 1 PN" "C2905415" (at 293.37 129.54 0)
+    (property "Distributor 1 PN" "C6332197" (at 293.37 129.54 0)
       (effects (font (size 1.27 1.27)) hide)
     )
-    (property "MPN" "KH-2.54FH-1X4P-H8.5" (at 293.37 129.54 0)
+    (property "MPN" "HB-PH3-25414PB2GOP" (at 293.37 129.54 0)
       (effects (font (size 1.27 1.27)) hide)
     )
-    (property "Manufacturer" "Shenzhen Kinghelm Elec" (at 293.37 129.54 0)
+    (property "Manufacturer" "Hanbo Electronic" (at 293.37 129.54 0)
       (effects (font (size 1.27 1.27)) hide)
     )
