File: elec/Control Board/Control_1v1/Control_1v1/SPI_ControllerLevel_Shifter.kicad_sch (KiCad schematic)
At the start: 34 parts, among them J301 RJ12_6P6C_HORZ, J302 0.100_2Pin, Q301 BSS138, Q302 BSS138, Q303 BSS138, Q304 BSS138

Commit message: Add JLCPCB order files after fixing out of stock components.
Parts:
- J301: Distributor 1 PN C305981 -> C2683355
Changed lines of the file:
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@@
       (effects (font (size 1.27 1.27)) hide)
     )
-    (property "Distributor 1 PN" "C305981" (at 116.84 137.16 0)
+    (property "Distributor 1 PN" "C2683355" (at 116.84 137.16 0)
       (effects (font (size 1.27 1.27)) hide)
     )
