File: elec/Control Board/Control_1v1/Control_1v1/Adafruit-MAX31850-thermocouple-breakout-board.kicad_sch (KiCad schematic)
At the start: 37 parts, among them J11 Screw_Terminal_01x02, J2 MAX31850K

Commit message: Add JLCPCB order files after fixing out of stock components.
Parts:
- R203: Distributor 1 PN C269713 -> C23162; Manufacturer TyoHM -> UNI-ROYAL(Uniroyal Elec)
Changed lines of the file:
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@@
       (effects (font (size 1.27 1.27)) hide)
     )
-    (property "Distributor 1 PN" "C269713" (at 207.01 167.64 90)
+    (property "Distributor 1 PN" "C23162" (at 207.01 167.64 90)
       (effects (font (size 1.27 1.27)) hide)
     )
-    (property "Manufacturer" "TyoHM" (at 207.01 167.64 90)
+    (property "Manufacturer" "UNI-ROYAL(Uniroyal Elec)" (at 207.01 167.64 90)
       (effects (font (size 1.27 1.27)) hide)
     )
@@
       (effects (font (size 1.27 1.27)) hide)
     )
-    (property "Description" "1W ±1% 4.7kΩ 0603 Chip Resistor - Surface Mount ROHS" (at 207.01 167.64 0)
+    (property "Description" "100mW Thick Film Resistors ±100ppm/℃ ±1% 4.7kΩ 0603 Chip Resistor - Surface Mount ROHS" (at 207.01 167.64 0)
       (effects (font (size 1.27 1.27)) hide)
     )

Commit message: Changes to change headders to sockets. Scockets for thermcouple amplifiers.
Parts:
- J2, JP10, JP15: Distributor 1 adafruit -> JLCPCB; Distributor 1 PN 1727 -> C2905417
Changed lines of the file:
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@@
       (effects (font (size 1.27 1.27)) hide)
     )
-    (property "Description" "1x2P 20A -40℃~+105℃ 300V Green 12~30 Straight pin 5.08mm 2.5 1 2 Plugin,P=5.08mm Screw terminal ROHS" (at 345.44 171.45 0)
+    (property "Description" "1x2P XH 1 2.5mm 2 Brass Plugin,P=2.5mm Wire To Board / Wire To Wire Connector ROHS" (at 345.44 171.45 0)
       (effects (font (size 1.27 1.27)) hide)
     )
@@
       (effects (font (size 1.27 1.27)) hide)
     )
-    (property "Description" "1x2P 20A -40℃~+105℃ 300V Green 12~30 Straight pin 5.08mm 2.5 1 2 Plugin,P=5.08mm Screw terminal ROHS" (at 191.77 223.52 0)
+    (property "Description" "1x2P XH 1 2.5mm 2 Brass Plugin,P=2.5mm Wire To Board / Wire To Wire Connector ROHS" (at 191.77 223.52 0)
       (effects (font (size 1.27 1.27)) hide)
     )
@@
       (effects (font (size 1.27 1.27)) hide)
     )
-    (property "Description" "Thermocouple Amplifier with 1-Wire Breakout Board - MAX31850K" (at 176.53 137.16 0)
-      (effects (font (size 1.27 1.27)) hide)
-    )
-    (property "Distributor 1" "adafruit" (at 176.53 137.16 0)
-      (effects (font (size 1.27 1.27)) hide)
-    )
-    (property "Distributor 1 PN" "1727" (at 176.53 137.16 0)
+    (property "Description" "2.54mm Plugin 3A 8P -40℃~+105℃ Straight 1x8P 8.5mm Top Square Holes Plugin,P=2.54mm Female Headers ROHS" (at 176.53 137.16 0)
+      (effects (font (size 1.27 1.27)) hide)
+    )
+    (property "Distributor 1" "JLCPCB" (at 176.53 137.16 0)
+      (effects (font (size 1.27 1.27)) hide)
+    )
+    (property "Distributor 1 PN" "C2905417" (at 176.53 137.16 0)
       (effects (font (size 1.27 1.27)) hide)
     )
@@
       (effects (font (size 1.27 1.27)) hide)
     )
-    (property "Description" "1x2P 20A -40℃~+105℃ 300V Green 12~30 Straight pin 5.08mm 2.5 1 2 Plugin,P=5.08mm Screw terminal ROHS" (at 181.61 156.21 0)
+    (property "Description" "1x2P XH 1 2.5mm 2 Brass Plugin,P=2.5mm Wire To Board / Wire To Wire Connector ROHS" (at 181.61 156.21 0)
       (effects (font (size 1.27 1.27)) hide)
     )
@@
       (effects (font (size 1.27 1.27)) hide)
     )
-    (property "Description" "Thermocouple Amplifier with 1-Wire Breakout Board - MAX31850K" (at 198.12 196.85 0)
-      (effects (font (size 1.27 1.27)) hide)
-    )
-    (property "Distributor 1" "adafruit" (at 198.12 196.85 0)
-      (effects (font (size 1.27 1.27)) hide)
-    )
-    (property "Distributor 1 PN" "1727" (at 198.12 196.85 0)
+    (property "Description" "2.54mm Plugin 3A 8P -40℃~+105℃ Straight 1x8P 8.5mm Top Square Holes Plugin,P=2.54mm Female Headers ROHS" (at 198.12 196.85 0)
+      (effects (font (size 1.27 1.27)) hide)
+    )
+    (property "Distributor 1" "JLCPCB" (at 198.12 196.85 0)
+      (effects (font (size 1.27 1.27)) hide)
+    )
+    (property "Distributor 1 PN" "C2905417" (at 198.12 196.85 0)
       (effects (font (size 1.27 1.27)) hide)
     )
@@
       (effects (font (size 1.27 1.27)) hide)
     )
-    (property "Description" "Thermocouple Amplifier with 1-Wire Breakout Board - MAX31850K" (at 342.9 143.51 0)
-      (effects (font (size 1.27 1.27)) hide)
-    )
-    (property "Distributor 1" "adafruit" (at 342.9 143.51 0)
-      (effects (font (size 1.27 1.27)) hide)
-    )
-    (property "Distributor 1 PN" "1727" (at 342.9 143.51 0)
-      (effects (font (size 1.27 1.27)) hide)
-    )
+    (property "Description" "2.54mm Plugin 3A 8P -40℃~+105℃ Straight 1x8P 8.5mm Top Square Holes Plugin,P=2.54mm Female Headers ROHS" (at 342.9 143.51 0)
+      (effects (font (size 1.27 1.27)) hide)
+    )
+    (property "Distributor 1" "JLCPCB" (at 342.9 143.51 0)
+      (effects (font (size 1.27 1.27)) hide)
+    )
+    (property "Distributor 1 PN" "C2905417" (at 342.9 143.51 0)
+      (effects (font (size 1.27 1.27)) hide)
+    )
