File: elec/Control Board/Control_1v1/Control_1v1/Adafruit-MAX31856-PCB-master.kicad_sch (KiCad schematic)
At the start: 8 parts, among them J10 MCP9600, J8 MCP9600, J9 MCP9600

Commit message: Changes to change headders to sockets. Scockets for thermcouple amplifiers.
Parts:
- J10, J8, J9: Distributor 1 adafruit -> JLCPCB; Distributor 1 PN 4101 -> C2932673
Changed lines of the file:
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@@
       (effects (font (size 1.27 1.27)) hide)
     )
-    (property "Description" "Adafruit MCP9600 I2C Thermocouple Amplifier - K, J, T, N, S, E, B and R Type T" (at 161.29 77.47 0)
-      (effects (font (size 1.27 1.27)) hide)
-    )
-    (property "Distributor 1" "adafruit" (at 161.29 77.47 0)
-      (effects (font (size 1.27 1.27)) hide)
-    )
-    (property "Distributor 1 PN" "4101" (at 161.29 77.47 0)
+    (property "Description" "2.54mm Plugin 3A 9P -40℃~+105℃ Straight 1x9P 8.5mm Top Square Holes Plugin,P=2.54mm Female Headers ROHS" (at 161.29 77.47 0)
+      (effects (font (size 1.27 1.27)) hide)
+    )
+    (property "Distributor 1" "JLCPCB" (at 161.29 77.47 0)
+      (effects (font (size 1.27 1.27)) hide)
+    )
+    (property "Distributor 1 PN" "C2932673" (at 161.29 77.47 0)
       (effects (font (size 1.27 1.27)) hide)
     )
@@
       (effects (font (size 1.27 1.27)) hide)
     )
-    (property "Description" "Adafruit MCP9600 I2C Thermocouple Amplifier - K, J, T, N, S, E, B and R Type T" (at 138.43 77.47 0)
-      (effects (font (size 1.27 1.27)) hide)
-    )
-    (property "Distributor 1" "adafruit" (at 138.43 77.47 0)
-      (effects (font (size 1.27 1.27)) hide)
-    )
-    (property "Distributor 1 PN" "4101" (at 138.43 77.47 0)
+    (property "Description" "2.54mm Plugin 3A 9P -40℃~+105℃ Straight 1x9P 8.5mm Top Square Holes Plugin,P=2.54mm Female Headers ROHS" (at 138.43 77.47 0)
+      (effects (font (size 1.27 1.27)) hide)
+    )
+    (property "Distributor 1" "JLCPCB" (at 138.43 77.47 0)
+      (effects (font (size 1.27 1.27)) hide)
+    )
+    (property "Distributor 1 PN" "C2932673" (at 138.43 77.47 0)
       (effects (font (size 1.27 1.27)) hide)
     )
@@
       (effects (font (size 1.27 1.27)) hide)
     )
-    (property "Description" "Adafruit MCP9600 I2C Thermocouple Amplifier - K, J, T, N, S, E, B and R Type T" (at 115.57 77.47 0)
-      (effects (font (size 1.27 1.27)) hide)
-    )
-    (property "Distributor 1" "adafruit" (at 115.57 77.47 0)
-      (effects (font (size 1.27 1.27)) hide)
-    )
-    (property "Distributor 1 PN" "4101" (at 115.57 77.47 0)
-      (effects (font (size 1.27 1.27)) hide)
-    )
+    (property "Description" "2.54mm Plugin 3A 9P -40℃~+105℃ Straight 1x9P 8.5mm Top Square Holes Plugin,P=2.54mm Female Headers ROHS" (at 115.57 77.47 0)
+      (effects (font (size 1.27 1.27)) hide)
+    )
+    (property "Distributor 1" "JLCPCB" (at 115.57 77.47 0)
+      (effects (font (size 1.27 1.27)) hide)
+    )
+    (property "Distributor 1 PN" "C2932673" (at 115.57 77.47 0)
+      (effects (font (size 1.27 1.27)) hide)
+    )
