File: elec/Control Board/Control_1v1/Control_1v1/Fan controller.kicad_sch (KiCad schematic)
At the start: 37 parts, among them J10 Conn_01x05, J11 Conn_01x04, J12 Conn_01x07, J20 Conn_01x04, J6 DB25_Female_MountingHoles, J9 Conn_01x04, Q2 NCE01P30K, Q601 BSS138

Commit message: Move components away from J35, J36.
Parts:
- J11, J20, J9: Distributor 1 PN C2905415 -> C6332197; MPN KH-2.54FH-1X4P-H8.5 -> HB-PH3-25414PB2GOP; Manufacturer Shenzhen Kinghelm Elec -> Hanbo Electronic
Changed lines of the file:
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@@
       (effects (font (size 1.27 1.27)) hide)
     )
-    (property "Datasheet" "KH-2.54FH-1X4P-H8.5.pdf" (at 165.1 121.92 0)
+    (property "Datasheet" "HB-PH3-25414PB2GOP.pdf" (at 165.1 121.92 0)
       (effects (font (size 1.27 1.27)) hide)
     )
@@
       (effects (font (size 1.27 1.27)) hide)
     )
-    (property "Distributor 1 PN" "C2905415" (at 165.1 121.92 0)
-      (effects (font (size 1.27 1.27)) hide)
-    )
-    (property "MPN" "KH-2.54FH-1X4P-H8.5" (at 165.1 121.92 0)
-      (effects (font (size 1.27 1.27)) hide)
-    )
-    (property "Manufacturer" "Shenzhen Kinghelm Elec" (at 165.1 121.92 0)
+    (property "Distributor 1 PN" "C6332197" (at 165.1 121.92 0)
+      (effects (font (size 1.27 1.27)) hide)
+    )
+    (property "MPN" "HB-PH3-25414PB2GOP" (at 165.1 121.92 0)
+      (effects (font (size 1.27 1.27)) hide)
+    )
+    (property "Manufacturer" "Hanbo Electronic" (at 165.1 121.92 0)
       (effects (font (size 1.27 1.27)) hide)
     )
@@
       (effects (font (size 1.27 1.27)) hide)
     )
-    (property "Datasheet" "KH-2.54FH-1X4P-H8.5.pdf" (at 220.98 81.28 0)
+    (property "Datasheet" "HB-PH3-25414PB2GOP.pdf" (at 220.98 81.28 0)
       (effects (font (size 1.27 1.27)) hide)
     )
@@
       (effects (font (size 1.27 1.27)) hide)
     )
-    (property "Distributor 1 PN" "C2905415" (at 220.98 81.28 0)
-      (effects (font (size 1.27 1.27)) hide)
-    )
-    (property "MPN" "KH-2.54FH-1X4P-H8.5" (at 220.98 81.28 0)
-      (effects (font (size 1.27 1.27)) hide)
-    )
-    (property "Manufacturer" "Shenzhen Kinghelm Elec" (at 220.98 81.28 0)
+    (property "Distributor 1 PN" "C6332197" (at 220.98 81.28 0)
+      (effects (font (size 1.27 1.27)) hide)
+    )
+    (property "MPN" "HB-PH3-25414PB2GOP" (at 220.98 81.28 0)
+      (effects (font (size 1.27 1.27)) hide)
+    )
+    (property "Manufacturer" "Hanbo Electronic" (at 220.98 81.28 0)
       (effects (font (size 1.27 1.27)) hide)
     )
@@
       (effects (font (size 1.27 1.27)) hide)
     )
-    (property "Datasheet" "KH-2.54FH-1X4P-H8.5.pdf" (at 177.8 100.33 0)
+    (property "Datasheet" "HB-PH3-25414PB2GOP.pdf" (at 177.8 100.33 0)
       (effects (font (size 1.27 1.27)) hide)
     )
@@
       (effects (font (size 1.27 1.27)) hide)
     )
-    (property "Distributor 1 PN" "C2905415" (at 177.8 100.33 0)
-      (effects (font (size 1.27 1.27)) hide)
-    )
-    (property "MPN" "KH-2.54FH-1X4P-H8.5" (at 177.8 100.33 0)
-      (effects (font (size 1.27 1.27)) hide)
-    )
-    (property "Manufacturer" "Shenzhen Kinghelm Elec" (at 177.8 100.33 0)
-      (effects (font (size 1.27 1.27)) hide)
-    )
+    (property "Distributor 1 PN" "C6332197" (at 177.8 100.33 0)
+      (effects (font (size 1.27 1.27)) hide)
+    )
+    (property "MPN" "HB-PH3-25414PB2GOP" (at 177.8 100.33 0)
+      (effects (font (size 1.27 1.27)) hide)
+    )
+    (property "Manufacturer" "Hanbo Electronic" (at 177.8 100.33 0)
+      (effects (font (size 1.27 1.27)) hide)
+    )

Commit message: Update Zener diode part number from MELF to miniMELF.
Parts:
- D1, D2: Cost 0.0433 -> 0.0097; MPN DL4733A -> ZMM5231; Manufacturer LGE -> JSMSEMI
Changed lines of the file:
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@@
       (effects (font (size 1.27 1.27)) hide)
     )
-    (property "Cost" "0.0433" (at 250.19 91.44 0)
+    (property "Cost" "0.0097" (at 250.19 91.44 0)
       (effects (font (size 1.27 1.27)) hide)
     )
-    (property "Description" "±5% Single 1W 5.1V MELF Zener Diodes ROHS" (at 250.19 91.44 0)
+    (property "Description" "±5% 500mW 5.1V MiniMELF(SOD-80) Zener Diodes ROHS" (at 250.19 91.44 0)
       (effects (font (size 1.27 1.27)) hide)
     )
@@
       (effects (font (size 1.27 1.27)) hide)
     )
-    (property "MPN" "DL4733A" (at 250.19 91.44 0)
+    (property "MPN" "ZMM5231" (at 250.19 91.44 0)
       (effects (font (size 1.27 1.27)) hide)
     )
-    (property "Manufacturer" "LGE" (at 250.19 91.44 0)
+    (property "Manufacturer" "JSMSEMI" (at 250.19 91.44 0)
       (effects (font (size 1.27 1.27)) hide)
     )
@@
       (effects (font (size 1.27 1.27)) hide)
     )
-    (property "Cost" "0.0433" (at 265.43 144.78 0)
+    (property "Cost" "0.0097" (at 265.43 144.78 0)
       (effects (font (size 1.27 1.27)) hide)
     )
-    (property "Description" "±5% Single 1W 5.1V MELF Zener Diodes ROHS" (at 265.43 144.78 0)
+    (property "Description" "±5% 500mW 5.1V MiniMELF(SOD-80) Zener Diodes ROHS" (at 265.43 144.78 0)
       (effects (font (size 1.27 1.27)) hide)
     )
@@
       (effects (font (size 1.27 1.27)) hide)
     )
-    (property "MPN" "DL4733A" (at 265.43 144.78 0)
+    (property "MPN" "ZMM5231" (at 265.43 144.78 0)
       (effects (font (size 1.27 1.27)) hide)
     )
-    (property "Manufacturer" "LGE" (at 265.43 144.78 0)
+    (property "Manufacturer" "JSMSEMI" (at 265.43 144.78 0)
       (effects (font (size 1.27 1.27)) hide)
     )
